File: maskmeter.kicad_pcb (KiCad board)
At the start: 2 copper layers, 41 x 37 mm, 12 parts, among them SW1 SW_Push, U1 TLC555IDR

Commit message: Updated battery holder
Parts:
- BT1: footprint maskmeter:QJ.BS-6 -> Battery:BatteryHolder_Keystone_1060_1x2032
- C1: value 10uF -> 0.1uF
- moved BT1 0.90 mm to (130.0, 90.6), turned to 270 degrees
Routing:
- net Net-(BT1-Pad1): track 25.2 -> 26.1 mm
Changed lines of the file:
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@@
   (general
     (thickness 1.6)
-    (drawings 21)
-    (tracks 65)
+    (drawings 20)
+    (tracks 66)
     (zones 0)
     (modules 12)
@@
   (page A4)
   (layers
-    (0 F.Cu signal hide)
-    (31 B.Cu signal hide)
+    (0 F.Cu signal)
+    (31 B.Cu signal)
     (32 B.Adhes user)
     (33 F.Adhes user)
@@
     (add_net VCC)
   )
+  (module Battery:BatteryHolder_Keystone_1060_1x2032 (layer F.Cu)
+    (at 130 90.6 270)
+    (descr http://www.keyelco.com/product-pdf.cfm?p=726)
+    (tags "CR2032 BR2032 BatteryHolder Battery")
+    (attr smd)
+    (fp_text reference BT1 (at -14.125 -5.3 90) (layer F.SilkS)
+      (effects (font (size 1 1) (thickness 0.15)))
+    )
+    (fp_text value Battery_Cell (at 0 -11.75 90) (layer F.Fab)
+      (effects (font (size 1 1) (thickness 0.15)))
+    )
+    (fp_line (start -12 6) (end -14 6) (layer F.SilkS) (width 0.12))
+    (fp_line (start -13 5) (end -13 7) (layer F.SilkS) (width 0.12))
+    (fp_text user %R (at 0 0 90) (layer F.Fab)
+      (effects (font (size 1 1) (thickness 0.15)))
+    )
+    (fp_line (start 11.5 -8.5) (end 6.5 -8.5) (layer F.CrtYd) (width 0.05))
+    (fp_arc (start 0 0) (end 6.5 -8.5) (angle -74.81070976) (layer F.CrtYd) (width 0.05))
+    (fp_line (start 11.5 4) (end 11.5 8.5) (layer F.CrtYd) (width 0.05))
+    (fp_line (start 14.7 4) (end 11.5 4) (layer F.CrtYd) (width 0.05))
+    (fp_line (start 14.7 2.3) (end 14.7 4) (layer F.CrtYd) (width 0.05))
+    (fp_line (start 16.45 2.3) (end 14.7 2.3) (layer F.CrtYd) (width 0.05))
+    (fp_line (start 16.45 -2.3) (end 16.45 2.3) (layer F.CrtYd) (width 0.05))
+    (fp_line (start 14.7 -2.3) (end 16.45 -2.3) (layer F.CrtYd) (width 0.05))
+    (fp_line (start 14.7 -4) (end 14.7 -2.3) (layer F.CrtYd) (width 0.05))
+    (fp_line (start 11.5 -4) (end 14.7 -4) (layer F.CrtYd) (width 0.05))
+    (fp_line (start 11.5 -8.5) (end 11.5 -4) (layer F.CrtYd) (width 0.05))
+    (fp_line (start -11.5 -8.5) (end -6.5 -8.5) (layer F.CrtYd) (width 0.05))
+    (fp_line (start -11.5 -4) (end -11.5 -8.5) (layer F.CrtYd) (width 0.05))
+    (fp_line (start -14.7 -4) (end -11.5 -4) (layer F.CrtYd) (width 0.05))
+    (fp_line (start -14.7 -2.3) (end -14.7 -4) (layer F.CrtYd) (width 0.05))
+    (fp_line (start -14.7 -2.3) (end -16.45 -2.3) (layer F.CrtYd) (width 0.05))
+    (fp_line (start -16.45 2.3) (end -16.45 -2.3) (layer F.CrtYd) (width 0.05))
+    (fp_line (start -14.7 2.3) (end -16.45 2.3) (layer F.CrtYd) (width 0.05))
+    (fp_line (start -14.7 4) (end -14.7 2.3) (layer F.CrtYd) (width 0.05))
+    (fp_line (start -14.7 4) (end -11.5 4) (layer F.CrtYd) (width 0.05))
+    (fp_line (start -11.5 4) (end -11.5 8.5) (layer F.CrtYd) (width 0.05))
+    (fp_line (start -6.5 8.5) (end -11.5 8.5) (layer F.CrtYd) (width 0.05))
+    (fp_line (start 11.5 8.5) (end 6.5 8.5) (layer F.CrtYd) (width 0.05))
+    (fp_arc (start 0 0) (end -6.5 8.5) (angle -74.81070976) (layer F.CrtYd) (width 0.05))
+    (fp_line (start 11.35 -8.35) (end 11.35 -3.85) (layer F.SilkS) (width 0.12))
+    (fp_line (start -11.35 -8.35) (end -11.35 -3.85) (layer F.SilkS) (width 0.12))
+    (fp_line (start -11.35 -8.35) (end 11.35 -8.35) (layer F.SilkS) (width 0.12))
+    (fp_line (start 14.55 -3.85) (end 14.55 -2.3) (layer F.SilkS) (width 0.12))
+    (fp_line (start 11.35 -3.85) (end 14.55 -3.85) (layer F.SilkS) (width 0.12))
+    (fp_line (start -14.55 -3.85) (end -14.55 -2.3) (layer F.SilkS) (width 0.12))
+    (fp_line (start -11.35 -3.85) (end -14.55 -3.85) (layer F.SilkS) (width 0.12))
+    (fp_line (start -14.55 3.85) (end -14.55 2.3) (layer F.SilkS) (width 0.12))
+    (fp_line (start -11.35 3.85) (end -14.55 3.85) (layer F.SilkS) (width 0.12))
+    (fp_line (start -9.55 8.35) (end -11.35 6.55) (layer F.SilkS) (width 0.12))
+    (fp_line (start -11.35 6.55) (end -11.35 3.85) (layer F.SilkS) (width 0.12))
+    (fp_line (start 11.35 8.35) (end -9.55 8.35) (layer F.SilkS) (width 0.12))
+    (fp_line (start 11.35 8.35) (end 11.35 3.85) (layer F.SilkS) (width 0.12))
+    (fp_line (start 14.55 3.85) (end 14.55 2.3) (layer F.SilkS) (width 0.12))
+    (fp_line (start 11.35 3.85) (end 14.55 3.85) (layer F.SilkS) (width 0.12))
+    (fp_line (start -9.4 8) (end -11 6.4) (layer F.Fab) (width 0.1))
+    (fp_line (start 14.2 -3.5) (end 11 -3.5) (layer F.Fab) (width 0.1))
+    (fp_line (start 14.2 3.5) (end 14.2 -3.5) (layer F.Fab) (width 0.1))
+    (fp_line (start 11 3.5) (end 14.2 3.5) (layer F.Fab) (width 0.1))
+    (fp_line (start -14.2 -3.5) (end -11 -3.5) (layer F.Fab) (width 0.1))
+    (fp_line (start -14.2 3.5) (end -14.2 -3.5) (layer F.Fab) (width 0.1))
+    (fp_line (start -11 3.5) (end -14.2 3.5) (layer F.Fab) (width 0.1))
+    (fp_line (start -11 6.4) (end -11 3.5) (layer F.Fab) (width 0.1))
+    (fp_line (start -11 -8) (end -11 -3.5) (layer F.Fab) (width 0.1))
+    (fp_line (start 11 -8) (end 11 -3.5) (layer F.Fab) (width 0.1))
+    (fp_line (start 11 8) (end 11 3.5) (layer F.Fab) (width 0.1))
+    (fp_line (start 11 -8) (end -11 -8) (layer F.Fab) (width 0.1))
+    (fp_line (start 11 8) (end -9.4 8) (layer F.Fab) (width 0.1))
+    (fp_circle (center 0 0) (end -10.2 0) (layer Dwgs.User) (width 0.3))
+    (pad 1 smd rect (at -14.65 0 90) (size 2.6 3.6) (layers F.Cu F.Paste F.Mask)
+      (net 1 "Net-(BT1-Pad1)"))
+    (pad 2 smd rect (at 14.65 0 90) (size 2.6 3.6) (layers F.Cu F.Paste F.Mask)
+      (net 7 GND))
+    (model ${KISYS3DMOD}/Battery.3dshapes/BatteryHolder_Keystone_1060_1x2032.wrl
+      (at (xyz 0 0 0))
+      (scale (xyz 1 1 1))
+      (rotate (xyz 0 0 0))
+    )
+  )
   (module maskmeter:PCB_Resistance_Pad (layer B.Cu)
     (at 113.7 89.8)
@@
     (pad 2 smd rect (at -7.25 -5.75) (size 1.5 1.5) (layers B.Cu B.Mask)
       (net 6 "Net-(R3-Pad2)"))
-  )
-  (module maskmeter:QJ.BS-6 (layer F.Cu)
-    (at 129.1 90.6 180)
-    (fp_text reference BT1 (at -4.2 15.4) (layer F.SilkS)
-      (effects (font (size 1 1) (thickness 0.15)))
-    )
-    (fp_text value Battery_Cell (at 0.3 17.8) (layer F.Fab) hide
-      (effects (font (size 1 1) (thickness 0.15)))
-    )
-    (fp_line (start 3.5 -11.5) (end 10 -11.5) (layer F.CrtYd) (width 0.12))
-    (fp_line (start 3.5 -14.5) (end 3.5 -11.5) (layer F.CrtYd) (width 0.12))
-    (fp_line (start 2.5 -14.5) (end 3.5 -14.5) (layer F.CrtYd) (width 0.12))
-    (fp_line (start 10 10.5) (end 10 -11.5) (layer F.CrtYd) (width 0.12))
-    (fp_line (start 4 10.5) (end 10 10.5) (layer F.CrtYd) (width 0.12))
-    (fp_line (start 4 14.5) (end 4 10.5) (layer F.CrtYd) (width 0.12))
-    (fp_line (start 2.5 14.5) (end 4 14.5) (layer F.CrtYd) (width 0.12))
-    (fp_line (start -4 14.5) (end 2.5 14.5) (layer F.CrtYd) (width 0.12))
-    (fp_line (start -4 10.5) (end -4 14.5) (layer F.CrtYd) (width 0.12))
-    (fp_line (start -10 10.5) (end -4 10.5) (layer F.CrtYd) (width 0.12))
-    (fp_line (start -10 -11.5) (end -10 10.5) (layer F.CrtYd) (width 0.12))
-    (fp_line (start -3.5 -11.5) (end -10 -11.5) (layer F.CrtYd) (width 0.12))
-    (fp_line (start -3.5 -14.5) (end -3.5 -11.5) (layer F.CrtYd) (width 0.12))
-    (fp_line (start 2.5 -14.5) (end -3.5 -14.5) (layer F.CrtYd) (width 0.12))
-    (pad 2 smd rect (at 0 -14.5 180) (size 4.2 3) (layers F.Cu F.Paste F.Mask)
-      (net 7 GND))
-    (pad 1 smd rect (at 0 14.5 180) (size 4.2 3) (layers F.Cu F.Paste F.Mask)
-      (net 1 "Net-(BT1-Pad1)"))
   )
   (module Buzzer_Beeper:Buzzer_Murata_PKMCS0909E4000-R1 (layer F.Cu)
@@
       (effects (font (size 1 1) (thickness 0.15)))
     )
-    (fp_text value 10uF (at 0 1.43) (layer F.Fab)
+    (fp_text value 0.1uF (at 0 1.43) (layer F.Fab)
       (effects (font (size 1 1) (thickness 0.15)))
     )
@@
   (gr_arc (start 139 106) (end 139 109) (angle -90) (layer Edge.Cuts) (width 0.1))
   (gr_arc (start 139 75) (end 142 75) (angle -90) (layer Edge.Cuts) (width 0.1))
-  (gr_circle (center 129.198165 90.4) (end 140.1 90.4) (layer F.SilkS) (width 0.2))
   (gr_line (start 142 106) (end 142 75) (layer Edge.Cuts) (width 0.1))
   (gr_line (start 101 75) (end 101 106) (layer Edge.Cuts) (width 0.1))
+  (segment (start 114.9 93.15) (end 114.9 86.85) (width 0.5) (layer F.Cu) (net 1))
   (segment (start 114.9 86.5) (end 114.9 86.85) (width 0.5) (layer F.Cu) (net 1))
   (segment (start 125.3 76.1) (end 114.9 86.5) (width 0.5) (layer F.Cu) (net 1))
-  (segment (start 129.1 76.1) (end 125.3 76.1) (width 0.5) (layer F.Cu) (net 1))
-  (segment (start 114.9 93.15) (end 114.9 86.85) (width 0.5) (layer F.Cu) (net 1))
+  (segment (start 129.85 76.1) (end 125.3 76.1) (width 0.5) (layer F.Cu) (net 1))
+  (segment (start 130 75.95) (end 129.85 76.1) (width 0.5) (layer F.Cu) (net 1))
   (segment (start 110 74.7) (end 107.735 76.965) (width 0.25) (layer F.Cu) (net 2))
   (segment (start 114.9125 78.1) (end 114.9125 76.3125) (width 0.25) (layer F.Cu) (net 2))
