File: pcb/maskmeter.kicad_pcb (KiCad board)
At the start: 2 copper layers, 41 x 37 mm, 12 parts, among them SW1 SW_Push, U1 TLC555IDR

Commit message: Changed resitors and green LED
Other:
- board text added: "Keep sensor area clean and dry"
- board text added: "Mask Moisture Meter Plase on face mask and press the button Solid green light => Mask dry Alternating green and red => Mask moist Faster blinking / higher pitch noise => More moisture"
- board text removed: "Keep sensor area clean"
- board text removed: "Mask Moisture Meter Plase on face mask and press the button Solid yellow light: Mask dry Alternating yellow and red: Mask moist Faster blinking = more moisture"
Changed lines of the file:
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@@
   (page A4)
   (layers
-    (0 F.Cu signal)
-    (31 B.Cu signal)
+    (0 F.Cu signal hide)
+    (31 B.Cu signal hide)
     (32 B.Adhes user)
     (33 F.Adhes user)
@@
     (35 F.Paste user)
     (36 B.SilkS user)
-    (37 F.SilkS user)
+    (37 F.SilkS user hide)
     (38 B.Mask user)
     (39 F.Mask user)
@@
     )
   )
-  (gr_text "Keep sensor area clean" (at 123.5 90.8 270) (layer B.SilkS)
+  (gr_text "Keep sensor area clean and dry" (at 123.5 90.8 270) (layer B.SilkS)
     (effects (font (size 1 1) (thickness 0.15)) (justify mirror))
   )
-  (gr_text "Mask Moisture Meter\n\nPlase on face mask and press the button\nSolid yellow light: Mask dry\nAlternating yellow and red: Mask moist\nFaster blinking = more moisture" (at 133.2 106.6 270) (layer B.SilkS)
+  (gr_text "Mask Moisture Meter\n\nPlase on face mask and press the button\n\nSolid green light => Mask dry\nAlternating green and red => Mask moist\n\nFaster blinking / higher pitch noise \n=> More moisture" (at 133.2 106.6 270) (layer B.SilkS)
     (effects (font (size 1 1) (thickness 0.15)) (justify left mirror))
   )

Commit message: Set PCB thickness to 1mm
Other:
- net class  Power removed
- net class Default removed

Commit message: Revert "Set PCB thickness to 1mm"
This reverts commit 019fabce52c92cc1307a1fe131da5ab49f218db2.
Other:
- net class  Power added: clearance 0.2, trace_width 0.5, via_dia 0.8, via_drill 0.4
- net class Default added: clearance 0.2, trace_width 0.25, via_dia 0.8, via_drill 0.4
